Commit message: update camera_rgb and laser orientation

File: src/mxck_run/urdf/mxcarkit.urdf (robot description, URDF)
Before this commit: robot mxcarkit, 14 links, 13 joints
Links:
- removed link camera_link_1
- removed link lidar_link_1
- added link camera_rgb; visual box size=0 0 0
- added link laser; visual box size=0 0 0
Joints:
- joint camera_joint: child camera_link_1 -> camera_rgb; origin xyz=0.19 0 0.116 rpy=0 0 0 -> xyz=0.19 0.06 0.116 rpy=-1.5708 0 -1.5708
- joint lidar_joint: child lidar_link_1 -> laser; origin xyz=0.1915 0 0.0865 rpy=0 0 0 -> xyz=0.1915 0 0.0865 rpy=0 0 3.1415

Commit message: update lidar position

File: src/mxck_run/urdf/mxcarkit.urdf (robot description, URDF)
Before this commit: robot mxcarkit, 14 links, 13 joints
Joints:
- joint lidar_joint: origin xyz=0.1915 0 0.0865 rpy=0 0 3.1415 -> xyz=0.1915 0 0.0865 rpy=0 0 3.9270
